File: 02-hardware/esc_brushless/_autosave-esc_brushless.sch (KiCad schematic (older format))
At the start: 15 parts, among them J1 Conn_HE13_1x1_5.08V, J2 Conn_HE13_1x1_5.08V, J3 DNP, J4 DNP, J5 Conn_HE13_1x2_2.54V, J6 DNP, J7 DNP, J8 DNP

Commit message: start routing
Parts:
- J3, J4: symbol esc_brushless-rescue:Conn_HE13_1x3_2.54-p_Misc -> esc_brushless-rescue:Conn_HE13_1x3_2.54-p_Misc-esc_brushless-rescue
Changed lines of the file:
@@
 $EndComp
 $Comp
-L esc_brushless-rescue:Conn_HE13_1x3_2.54-p_Misc J4
+L esc_brushless-rescue:Conn_HE13_1x3_2.54-p_Misc-esc_brushless-rescue J4
 U 1 1 608FE3F3
 P 1000 3850
@@
 $EndComp
 $Comp
-L esc_brushless-rescue:Conn_HE13_1x3_2.54-p_Misc J3
+L esc_brushless-rescue:Conn_HE13_1x3_2.54-p_Misc-esc_brushless-rescue J3
 U 1 1 6090DE8C
 P 1000 2900
