File: 02-hardware/esc_brushless/esc_brushless.kicad_pcb (KiCad board)
At the start: 4 copper layers, 50.8 x 33 mm, 100 parts, among them J1 Conn_HE13_1x1_5.08V, J2 Conn_HE13_1x1_5.08V, J3 DNP, J4 DNP, J5 Conn_HE13_1x2_2.54V, J6 DNP, J7 DNP, J8 DNP, Q1 IPD30N03S4L_09, Q2 IPD30N03S4L_09, Q3 IPD30N03S4L_09, Q4 IPD30N03S4L_09, Q5 IPD30N03S4L_09, Q6 IPD30N03S4L_09, Q7 BC848B, Q8 2SK1829, U1 DRV8301, U2 STM32G030_C8, U3 LDLN025M15R, U4 MAX487CSA_ESA

Commit message: PCB v1.0
Parts:
- removed J3: DNP, p_Package_Misc:PinHeader_1x03_P2.54mm_Vertical
- removed R7: R_0603, p_Package_Resistor_SMD:R_0603_1608Metric_Pad0.98x0.95mm_HandSolder
- removed R8: R_CTN_0608, p_Package_Resistor_SMD:R_0603_1608Metric_Pad0.98x0.95mm_HandSolder
- added TP3: test_point, p_Package_Misc:TP_SMD_1.25mm, B.Cu at (200.4, 103.1)
- C13, C14, C33, D1, D3, R1, R2, R26, R28, R29, R30, R31, R43, R44, TP1, U2: moved to F.Cu
- C15, C16, C2, C21, C23, C24, C9, D2, L1: moved to B.Cu
- R18, R19: value R_0603 -> R_shunt_2512; footprint p_Package_Resistor_SMD:R_0603_1608Metric_Pad0.98x0.95mm_HandSolder -> p_Package_Resistor_SMD:R_2512_6332Metric_shunt; moved to B.Cu
- moved R9 87.8 mm to (233.2, 118.9)
- moved J2 79.9 mm to (192.3, 116.2)
- moved C6 79.3 mm to (247.8, 116.8), turned to 90 degrees
- moved R2 79.2 mm to (207.3, 117.5), turned to 0 degrees
- moved D1 79.0 mm to (204.0, 117.5)
- moved C30 77.8 mm to (197.2, 99.2)
- moved C3 76.3 mm to (247.0, 112.1), turned to 90 degrees
- moved R20 76.2 mm to (246.0, 116.6), turned to 90 degrees
- moved R21 76.0 mm to (249.6, 116.6), turned to 270 degrees
- moved Q2 75.6 mm to (238.5, 114.3)
- moved Q1 75.5 mm to (238.5, 114.3), turned to 0 degrees
- moved R42 75.4 mm to (195.7, 99.2), turned to 270 degrees
- moved R38 75.2 mm to (202.4, 102.5), turned to 270 degrees
- moved R15 75.0 mm to (229.2, 105.7), turned to 90 degrees
- moved C1 75.0 mm to (226.4, 114.6), turned to 270 degrees
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Connections:
- C1 pad 1: /mos drive stage/SL_A -> /mos drive stage/SN1
- C1 pad 2: GND -> /mos drive stage/SP1
- C2 pad 1: /mos drive stage/SL_B -> /mos drive stage/SN2
- C2 pad 2: GND -> /mos drive stage/SP2
- C7 pad 1: /mos power stage/ADC_B -> /microcontroller/ADC_B
- C8 pad 1: /microcontroller/ADC_B -> /microcontroller/ADC_C
- R18 pad 1: GND -> /mos drive stage/SL_A
- R18 pad 2: /mos drive stage/SL_A -> GND
- R19 pad 1: GND -> /mos drive stage/SL_B
- R19 pad 2: /mos drive stage/SL_B -> GND
- R22 pad 1: /mos power stage/ADC_B -> /microcontroller/ADC_B
- R23 pad 2: /mos power stage/ADC_B -> /microcontroller/ADC_B
- R24 pad 1: /microcontroller/ADC_B -> /microcontroller/ADC_C
- R25 pad 2: /microcontroller/ADC_B -> /microcontroller/ADC_C
- TP2 pad 1: Net-(TP2-Pad1) -> /microcontroller/SW_DIO
- U1 pad 10: /microcontroller/SPI_CS -> /microcontroller/SPI_MISO
- U1 pad 30: GND -> /mos drive stage/SP2
- U1 pad 31: /mos drive stage/SL_B -> /mos drive stage/SN2
- U1 pad 32: GND -> /mos drive stage/SP1
- U1 pad 33: /mos drive stage/SL_A -> /mos drive stage/SN1
- U1 pad 55: (no net) -> Net-(U1-Pad55)
- U2 pad 1: /microcontroller/LED -> Net-(U2-Pad1)
- U2 pad 10: (no net) -> Net-(U2-Pad10)
- U2 pad 11: /microcontroller/SO1 -> /microcontroller/ADC_PVDD
- U2 pad 12: /microcontroller/SO2 -> Net-(U2-Pad12)
- U2 pad 13: /microcontroller/ADC_PVDD -> /RS488_phy/RS485_TX
- U2 pad 14: /SENSOR_1 -> /RS488_phy/RS485_RX
- U2 pad 15: /microcontroller/SPI_CS -> /RS488_phy/\RS485_RE
- U2 pad 16: /mos drive stage/SPI_CLK -> /RS488_phy/RS485_DE
- U2 pad 17: /microcontroller/SPI_CS -> Net-(U2-Pad17)
- U2 pad 18: /microcontroller/SPI_MOSI -> /microcontroller/LED
- U2 pad 19: /mos power stage/ADC_B -> /microcontroller/ADC_A
- U2 pad 2: (no net) -> Net-(U2-Pad2)
- U2 pad 21: /microcontroller/ADC_A -> /microcontroller/ADC_C
- U2 pad 22: /SENSOR_2 -> /SENSOR_1
- U2 pad 23: /RS488_phy/RS485_DE -> /microcontroller/SO2
- U2 pad 24: /RS488_phy/\RS485_RE -> /microcontroller/SO1
- U2 pad 25: /microcontroller/INL_A -> /microcontroller/INL_C
- U2 pad 27: /microcontroller/INL_C -> /microcontroller/INL_A
- U2 pad 28: /microcontroller/INH_A -> /microcontroller/INH_C
- U2 pad 3: (no net) -> Net-(U2-Pad3)
- U2 pad 30: /microcontroller/EN_GATE -> Net-(U2-Pad30)
- U2 pad 31: /microcontroller/DC_CAL -> Net-(U2-Pad31)
- U2 pad 32: /microcontroller/INH_C -> /microcontroller/INH_A
- U2 pad 33: (no net) -> /microcontroller/EN_GATE
- U2 pad 34: Net-(TP1-Pad1) -> /microcontroller/DC_CAL
- U2 pad 37: Net-(TP2-Pad1) -> /microcontroller/PWM
- U2 pad 38: /microcontroller/\PWRGD_FLT -> /microcontroller/\MCU_RST
- U2 pad 39: /microcontroller/\OVR_CUR_FLT -> Net-(U2-Pad39)
- U2 pad 40: /microcontroller/\FLT -> Net-(U2-Pad40)
- U2 pad 41: (no net) -> Net-(TP1-Pad1)
- U2 pad 42: /microcontroller/\MCU_RST -> /mos drive stage/SPI_CLK
- U2 pad 43: (no net) -> /microcontroller/SPI_MISO
- U2 pad 44: (no net) -> /microcontroller/SPI_MOSI
- U2 pad 45: /RS488_phy/RS485_TX -> /microcontroller/SPI_CS
- U2 pad 46: /RS488_phy/RS485_RX -> /microcontroller/\PWRGD_FLT
- U2 pad 47: (no net) -> /microcontroller/\OVR_CUR_FLT
- U2 pad 48: /microcontroller/PWM -> /microcontroller/\FLT
- U2 pad 8: (no net) -> Net-(U2-Pad8)
- U2 pad 9: (no net) -> Net-(U2-Pad9)
- U3 pad 4: (no net) -> Net-(U3-Pad4)
Routing:
- net +3V3: track 37.7 -> 130.7 mm, vias 7 -> 10
- net /microcontroller/ADC_C: track 0.00 -> 73.4 mm
- net /microcontroller/ADC_B: track 4.00 -> 67.5 mm
- net /microcontroller/ADC_A: track 4.01 -> 62.7 mm
- net /mos power stage/MOTOR_PH1: track 23.8 -> 78.8 mm, vias 0 -> 1
- net /mos drive stage/GL_C: track 0.00 -> 53.3 mm
- net GND: track 26.7 -> 73.7 mm, vias 23 -> 33
- net /mos power stage/MOTOR_PH3: track 33.5 -> 74.9 mm, vias 0 -> 1
- net /mos drive stage/GH_C: track 0.00 -> 39.2 mm, vias 0 -> 1
- net /SENSOR_1: track 1.84 -> 41.0 mm, vias 0 -> 1
- net /mos drive stage/GH_A: track 0.00 -> 32.2 mm, vias 0 -> 1
- net /mos drive stage/GH_B: track 0.00 -> 31.2 mm, vias 0 -> 1
- net /mos power stage/MOTOR_PH2: track 29.9 -> 59.6 mm, vias 0 -> 1
- net +5V: track 25.6 -> 54.1 mm, vias 6 -> 8
- net /microcontroller/\OVR_CUR_FLT: track 7.89 -> 35.9 mm, vias 1 -> 0
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- removed copper zone on Power, net +3V3
- removed copper zone on Power, net +5V
- removed copper zone on F.Cu, net /mos power stage/MOTOR_PH1
- removed copper zone on F.Cu, net /mos power stage/MOTOR_PH2
- removed copper zone on F.Cu, net /mos power stage/MOTOR_PH3
Other:
- board size 50.8 x 33 mm -> 64.6 x 29.8 mm
- net class JLCPCB: clearance 0.127 -> 0.2; trace_width 0.20066 -> 0.25; via_dia 0.6096 -> 0.6; via_drill 0.3048 -> 0.3
- rule trace_min: 0.2 -> 0.25
