File: 02-hardware/esc_brushless/esc_brushless.sch (KiCad schematic (older format))
At the start: 15 parts, among them J1 Conn_HE13_1x1_5.08V, J2 Conn_HE13_1x1_5.08V, J3 DNP, J4 DNP, J5 Conn_HE13_1x2_2.54V, J6 DNP, J7 DNP, J8 DNP

Commit message: PCB v1.0
Parts:
- removed J3: DNP, p_Package_Misc:PinHeader_1x03_P2.54mm_Vertical, symbol esc_brushless-rescue:Conn_HE13_1x3_2.54-p_Misc
- removed R7: R_0603, p_Package_Resistor_SMD:R_0603_1608Metric_Pad0.98x0.95mm_HandSolder, symbol p_Passive:R_0603
- removed R8: R_CTN_0608, p_Package_Resistor_SMD:R_0603_1608Metric_Pad0.98x0.95mm_HandSolder, symbol p_Passive:R_CTN_0608
- added TP2, TP3: test_point, p_Package_Misc:TP_SMD_1.25mm, symbol p_Misc:test_point
- J4: symbol esc_brushless-rescue:Conn_HE13_1x3_2.54-p_Misc -> esc_brushless-rescue:Conn_HE13_1x3_2.54-p_Misc-esc_brushless-rescue-esc_brushless-rescue
Connections:
- net labels removed: SENSOR_2
- wire segments 120 -> 112
Changed lines of the file:
@@
 F9 "SH_C" O L 7950 3650 50
 F10 "GL_C" I L 7950 3750 50
-F11 "ADC_C" O L 7950 5200 50
-F12 "ADC_B" O L 7950 5300 50
+F11 "ADC_C" O L 7950 5300 50
+F12 "ADC_B" O L 7950 5200 50
 F13 "ADC_A" O L 7950 5100 50
 F14 "V_PWR" I L 7950 1650 50
@@
 F34 "GND" U R 5450 5550 50
 F35 "TEMP_SENSOR1" I L 3700 4650 50
-F36 "TEMP_SENSOR2" I L 3700 4850 50
 $EndSheet
 $Sheet
@@
 $EndComp
 $Comp
-L esc_brushless-rescue:Conn_HE13_1x3_2.54-p_Misc J4
+L esc_brushless-rescue:Conn_HE13_1x3_2.54-p_Misc-esc_brushless-rescue-esc_brushless-rescue J4
 U 1 1 608FE3F3
 P 1000 3850
@@
 F 3 "" H 900 3850 50  0001 C CNN
 	1    1000 3850
-	-1   0    0    -1
-$EndComp
-$Comp
-L esc_brushless-rescue:Conn_HE13_1x3_2.54-p_Misc J3
-U 1 1 6090DE8C
-P 1000 2900
-F 0 "J3" H 1100 3150 50  0000 C CNN
-F 1 "DNP" H 1100 2550 50  0000 C CNN
-F 2 "p_Package_Misc:PinHeader_1x03_P2.54mm_Vertical" H 900 2900 50  0001 C CNN
-F 3 "" H 900 2900 50  0001 C CNN
-	1    1000 2900
 	-1   0    0    -1
 $EndComp
@@
 $EndComp
 $Comp
-L power:GND #PWR01
-U 1 1 60867B73
-P 1200 3200
-F 0 "#PWR01" H 1200 2950 50  0001 C CNN
-F 1 "GND" H 1205 3027 50  0000 C CNN
-F 2 "" H 1200 3200 50  0001 C CNN
-F 3 "" H 1200 3200 50  0001 C CNN
-	1    1200 3200
-	1    0    0    -1
-$EndComp
-$Comp
 L power:GND #PWR03
 U 1 1 60867F73
@@
 	1    0    0    -1
 $EndComp
-Wire Wire Line
-	1100 3050 1200 3050
-Wire Wire Line
-	1200 3050 1200 3200
 $Comp
 L power:GND #PWR02
@@
 Wire Notes Line width 12
 	700  3450 1950 3450
-Text Notes 1300 3150 0    50   ~ 0
-SWD connector
 Wire Notes Line width 12
 	1950 3450 1950 2500
@@
 	3300 5150 3300 6250
 $Comp
-L p_Passive:R_0603 R7
-U 1 1 60C62495
-P 5550 6550
-F 0 "R7" H 5450 6500 50  0000 C CNN
-F 1 "R_0603" H 5350 6600 50  0000 C CNN
-F 2 "p_Package_Resistor_SMD:R_0603_1608Metric_Pad0.98x0.95mm_HandSolder" H 5550 6550 50  0001 C CNN
-F 3 "" H 5550 6550 50  0001 C CNN
-	1    5550 6550
-	-1   0    0    1
-$EndComp
-$Comp
-L power:GND #PWR010
-U 1 1 60C77DC9
-P 5550 7150
-F 0 "#PWR010" H 5550 6900 50  0001 C CNN
-F 1 "GND" H 5555 6977 50  0000 C CNN
-F 2 "" H 5550 7150 50  0001 C CNN
-F 3 "" H 5550 7150 50  0001 C CNN
-	1    5550 7150
-	1    0    0    -1
-$EndComp
-Wire Wire Line
-	5550 7100 5550 7150
-$Comp
 L p_Passive:R_CTN_0608 R6
 U 1 1 60C86EDB
@@
 Text Label 4650 6750 0    50   ~ 0
 SENSOR_1
-Text Label 5750 6750 0    50   ~ 0
-SENSOR_2
-$Comp
-L p_Passive:R_CTN_0608 R8
-U 1 1 60CA5F49
-P 5550 6950
-F 0 "R8" H 5678 6996 50  0000 L CNN
-F 1 "R_CTN_0608" H 5678 6905 50  0000 L CNN
-F 2 "p_Package_Resistor_SMD:R_0603_1608Metric_Pad0.98x0.95mm_HandSolder" H 5550 6950 50  0001 C CNN
-F 3 "" H 5550 6950 50  0001 C CNN
-	1    5550 6950
-	1    0    0    -1
-$EndComp
-Wire Wire Line
-	5550 6700 5550 6750
-Wire Wire Line
-	5750 6750 5550 6750
-Connection ~ 5550 6750
-Wire Wire Line
-	5550 6750 5550 6800
 Wire Notes Line width 12
 	4000 6100 4000 7600
 Wire Notes Line width 12
-	6250 7600 6250 6100
-Wire Notes Line width 12
-	6250 6100 4000 6100
-Wire Notes Line width 12
-	4000 7600 6250 7600
-Text Notes 4750 7500 0    50   ~ 0
+	5200 7600 5200 6100
+Text Notes 4100 7500 0    50   ~ 0
 Temperature sensors
 Wire Wire Line
 	3700 4650 3100 4650
-Wire Wire Line
-	3700 4850 3100 4850
 Text Label 3100 4650 0    50   ~ 0
 SENSOR_1
-Text Label 3100 4850 0    50   ~ 0
-SENSOR_2
 $Comp
 L power:+5V #PWR0101
@@
 	5550 1750 5900 1750
 $Comp
-L power:+3.3V #PWR0110
-U 1 1 60ED6E72
-P 5550 6350
-F 0 "#PWR0110" H 5550 6200 50  0001 C CNN
-F 1 "+3.3V" H 5565 6523 50  0000 C CNN
-F 2 "" H 5550 6350 50  0001 C CNN
-F 3 "" H 5550 6350 50  0001 C CNN
-	1    5550 6350
-	1    0    0    -1
-$EndComp
-$Comp
 L power:+3.3V #PWR0111
 U 1 1 60ED8F6D
@@
 	1    0    0    -1
 $EndComp
-Wire Wire Line
-	5550 6350 5550 6400
 Wire Wire Line
 	4450 6350 4450 6400
@@
 	-1   0    0    1
 $EndComp
+$Comp
+L p_Misc:test_point TP2
+U 1 1 60A8B33B
+P 1000 2850
+F 0 "TP2" H 800 2850 50  0000 C CNN
+F 1 "test_point" H 987 2984 50  0001 C CNN
+F 2 "p_Package_Misc:TP_SMD_1.25mm" H 1000 2650 50  0001 C CNN
+F 3 "" H 1000 2850 50  0001 C CNN
+	1    1000 2850
+	1    0    0    -1
+$EndComp
+$Comp
+L p_Misc:test_point TP3
+U 1 1 60A8E4B3
+P 1000 2950
+F 0 "TP3" H 800 2950 50  0000 C CNN
+F 1 "test_point" H 987 3084 50  0001 C CNN
+F 2 "p_Package_Misc:TP_SMD_1.25mm" H 1000 2750 50  0001 C CNN
+F 3 "" H 1000 2950 50  0001 C CNN
+	1    1000 2950
+	1    0    0    -1
+$EndComp
+Text Notes 950  3100 0    50   ~ 0
+SWD connector
+Wire Notes Line width 12
+	5200 6100 4000 6100
+Wire Notes Line width 12
+	4000 7600 5200 7600
 $EndSCHEMATC
